Commit message: gazebo_ros2_control active

File: urdf/robot.urdf.xacro (robot description, xacro)
@@ -2,13 +2,9 @@
 <robot xmlns:xacro="http://www.ros.org/wiki/xacro"  name="diff_bot">
     <xacro:arg name="cmd_mode" default="position"/>
-    <xacro:arg name="real_time" default="true"/>
+    <xacro:arg name="HW_mode" default="mock"/>
     <xacro:include filename="robot_core.xacro"/>
-    <xacro:if value="$(arg real_time)">
-        <xacro:include filename="ros2_control.xacro"/>
-        <xacro:ros2_control cmd_mode="$(arg cmd_mode)"/>
-    </xacro:if>
-    <xacro:unless value="$(arg real_time)">
-        <xacro:include filename="sim_control.xacro"/>
-        <xacro:ros2_control_mock_hardware cmd_mode="$(arg cmd_mode)"/>
-    </xacro:unless>
+    <xacro:include filename="gazebo.xacro"/>
+    <xacro:include filename="ros2_control.xacro"/>
+    <!-- XACRO to handle multiple ros2_control hardware_interface plugins -->
+    <xacro:ros2_control HW_mode="$(arg HW_mode)" cmd_mode="$(arg cmd_mode)"/>
 </robot>

File: urdf/robot_core.xacro (robot description, xacro)
@@ -29,4 +29,9 @@
             </geometry>
         </collision>
+        <inertial>
+            <mass value="1.0"/>
+            <origin xyz="0 0 0" rpy="0 0 0"/>
+            <inertia ixx="0.01" ixy="0" ixz="0" iyy="0.01" iyz="0" izz="0.01"/>
+        </inertial>
     </link>
     <joint name="base_joint" type="fixed">
@@ -49,4 +54,9 @@
             </geometry>
         </collision>
+        <inertial>
+            <mass value="0.5"/>
+            <origin xyz="0 0 0" rpy="0 0 0"/>
+            <inertia ixx="0.01" ixy="0" ixz="0" iyy="0.01" iyz="0" izz="0.01"/>
+        </inertial>
     </link>
     <joint name="wrist_carrier_joint" type="revolute">
@@ -71,4 +81,9 @@
             </geometry>
         </collision>
+        <inertial>
+            <mass value="0.5"/>
+            <origin xyz="0 0 0" rpy="0 0 0"/>
+            <inertia ixx="0.01" ixy="0" ixz="0" iyy="0.01" iyz="0" izz="0.01"/>
+        </inertial>
     </link>
     <joint name="wrist_bevel_joint" type="revolute">

File: urdf/ros2_control.xacro (robot description, xacro)
@@ -1,36 +1,96 @@
 <?xml version="1.0"?>
 <robot xmlns:xacro="http://www.ros.org/wiki/xacro">
-    <xacro:macro name="ros2_control" params="cmd_mode">
-        <ros2_control name="StepperSystemHardware" type="system">
-            <hardware>
-                <plugin>diff_bot/StepperSystemHardware</plugin>
-                <param name="device">can0</param>
-                <param name="CAN_rate">500000</param>
-                <param name="timeout">5</param>
-                <param name="loop_rate">1000</param>
-            </hardware>
-            <joint name="wrist_carrier_joint">
-                <xacro:if value="${cmd_mode == 'position'}">
+    <xacro:macro name="ros2_control" params="HW_mode cmd_mode">
+        <xacro:if value="${HW_mode == 'real'}">
+            <ros2_control name="StepperSystemHardware" type="system">
+                <hardware>
+                    <plugin>diff_bot/StepperSystemHardware</plugin>
+                    <param name="device">can0</param>
+                    <param name="CAN_rate">500000</param>
+                    <param name="timeout">5</param>
+                    <param name="loop_rate">1000</param>
+                </hardware>
+                <joint name="wrist_carrier_joint">
+                    <xacro:if value="${cmd_mode == 'position'}">
+                        <command_interface name="position"/>
+                    </xacro:if>
+                    <command_interface name="velocity"/>
+                    <command_interface name="acceleration"/>
+                    <state_interface name="position"/>
+                    <state_interface name="velocity"/>
+                    <param name="reduction">2</param>
+                    <param name="CAN_id">0x01</param>
+                </joint>
+                <joint name="wrist_bevel_joint">
+                    <xacro:if value="${cmd_mode == 'position'}">
+                        <command_interface name="position"/>
+                    </xacro:if>
+                    <command_interface name="velocity"/>
+                    <command_interface name="acceleration"/>
+                    <state_interface name="position"/>
+                    <state_interface name="velocity"/>
+                    <param name="reduction">2</param>
+                    <param name="CAN_id">0x02</param>
+                </joint>
+            </ros2_control>
+        </xacro:if>
+        <xacro:if value="${HW_mode == 'gazebo'}">
+            <ros2_control name="GazeboSimSystem" type="system">
+                <hardware>
+                    <plugin>gazebo_ros2_control/GazeboSystem</plugin>
+                </hardware>
+                <joint name="wrist_carrier_joint">
+                    <xacro:if value="${cmd_mode == 'position'}">
                     <command_interface name="position"/>
-                </xacro:if>
-                <command_interface name="velocity"/>
-                <command_interface name="acceleration"/>
-                <state_interface name="position"/>
-                <state_interface name="velocity"/>
-                <param name="reduction">2</param>
-                <param name="CAN_id">0x01</param>
-            </joint>
-            <joint name="wrist_bevel_joint">
-                <xacro:if value="${cmd_mode == 'position'}">
+                    </xacro:if>
+                    <command_interface name="velocity"/>
+                    <!-- <command_interface name="acceleration"/> -->
+                    <state_interface name="position">
+                    <param name="initial_value">0.0</param>
+                    </state_interface>
+                    <state_interface name="velocity"/>
+                </joint>
+                <joint name="wrist_bevel_joint">
+                    <xacro:if value="${cmd_mode == 'position'}">
                     <command_interface name="position"/>
-                </xacro:if>
-                <command_interface name="velocity"/>
-                <command_interface name="acceleration"/>
-                <state_interface name="position"/>
-                <state_interface name="velocity"/>
-                <param name="reduction">2</param>
-                <param name="CAN_id">0x02</param>
-            </joint>
-        </ros2_control>
+                    </xacro:if>
+                    <command_interface name="velocity"/>
+                    <!-- <command_interface name="acceleration"/> -->
+                    <state_interface name="position">
+                    <param name="initial_value">0.0</param>
+                    </state_interface>
+                    <state_interface name="velocity"/>
+                </joint>
+            </ros2_control>
+        </xacro:if>
+        <xacro:if value="${HW_mode == 'mock'}">
+            <ros2_control name="sim_control" type="system">
+                <hardware>
+                    <plugin>mock_components/GenericSystem</plugin>
+                </hardware>
+                <joint name="wrist_carrier_joint">
+                    <xacro:if value="${cmd_mode == 'position'}">
+                    <command_interface name="position"/>
+                    </xacro:if>
+                    <command_interface name="velocity"/>
+                    <!-- <command_interface name="acceleration"/> -->
+                    <state_interface name="position">
+                    <param name="initial_value">0.0</param>
+                    </state_interface>
+                    <state_interface name="velocity"/>
+                </joint>
+                <joint name="wrist_bevel_joint">
+                    <xacro:if value="${cmd_mode == 'position'}">
+                    <command_interface name="position"/>
+                    </xacro:if>
+                    <command_interface name="velocity"/>
+                    <!-- <command_interface name="acceleration"/> -->
+                    <state_interface name="position">
+                    <param name="initial_value">0.0</param>
+                    </state_interface>
+                    <state_interface name="velocity"/>
+                </joint>
+            </ros2_control>
+        </xacro:if>
     </xacro:macro>
 </robot>
